Commit message: Add dynamical model of ARDrone

File: src/cognifli_simulator/cognifli_description/cognifli_drone/urdf/cognifli_drone.urdf.xacro (robot description, xacro)
@@ -1,211 +1,25 @@
 <?xml version="1.0"?>
-<robot name="lisa" xmlns:xacro="http://www.ros.org/wiki/xacro">
-  <xacro:include filename="$(find cognifli_description)/cognifli_drone/urdf/materials.xacro" />
-  <property name="M_PI" value="3.1415926535897931" />
-  <link name="base_footprint"/>
-  <!-- APM -->
-  <joint name="apm_joint" type="fixed">
-    <origin xyz="0 0 0" rpy="0 0 0" />
-    <parent link="base_link"/>
-    <child link="apm_link" />
-  </joint>
-  <link name="apm_link">
-    <inertial>
-      <origin xyz="0 0 0"/>
-      <mass value="0.01"/>
-      <inertia ixx="0.019995" ixy="0.0" ixz="0.0"
-               iyy="0.019995" iyz="0.0"
-               izz="0.03675" />
-    </inertial>
-  </link>
-  <!-- Wheel sensors -->
-  <joint name="encoder_joint" type="fixed">
-    <origin xyz="0 0 0" rpy="0 0 0" />
-    <parent link="base_link"/>
-    <child link="encoder_link" />
-  </joint>
-  <link name="encoder_link">
-    <inertial>
-      <origin xyz="0 0 0"/>
-      <mass value="0.01"/>
-      <inertia ixx="0.019995" ixy="0.0" ixz="0.0"
-               iyy="0.019995" iyz="0.0"
-               izz="0.03675" />
-    </inertial>
-  </link>
-  <joint name="base_joint" type="fixed">
-    <origin xyz="0 0 0.0102" rpy="0 0 0" />
-    <parent link="base_footprint"/>
-    <child link="base_link" />
-  </joint>
-  <link name="base_link">
-    <visual>
-      <geometry>
-        <cylinder length="0.10938" radius="0.178"/>
-      </geometry>
-      <origin xyz="0.001 0 0.05199" rpy="0 0 0"/>
-    </visual>
-    <collision>
-      <geometry>
-        <cylinder length="0.10938" radius="0.178"/>
-      </geometry>
-      <origin xyz="0.0 0 0.05949" rpy="0 0 0"/>
-    </collision>
-    <inertial>
-      <origin xyz="0.01 0 0"/>
-      <mass value="2.4"/>
-      <inertia ixx="0.019995" ixy="0.0" ixz="0.0"
-               iyy="0.019995" iyz="0.0"
-               izz="0.03675" />
-    </inertial>
-  </link>
-  <joint name="wheel_left_joint" type="fixed">
-    <parent link="base_link"/>
-    <child link="wheel_left_link"/>
-    <origin xyz="0.00 ${0.23/2} 0.0250" rpy="${-M_PI/2} 0 0"/>
-  </joint>
-  <link name="wheel_left_link">
-    <visual>
-      <geometry>
-        <cylinder length="0.0206" radius="0.0352"/>
-      </geometry>
-      <origin xyz="0 0 0" rpy="0 0 0"/>
-    </visual>
-    <collision>
-      <geometry>
-        <cylinder length="0.0206" radius="0.0352"/>
-      </geometry>
-      <origin rpy="0 0 0" xyz="0 0 0"/>
-    </collision>
-    <inertial>
-      <mass value="0.01" />
-      <origin xyz="0 0 0" />
-      <inertia ixx="0.001" ixy="0.0" ixz="0.0"
-               iyy="0.001" iyz="0.0"
-               izz="0.001" />
-    </inertial>
-  </link>
-  <joint name="wheel_right_joint" type="fixed">
-    <parent link="base_link"/>
-    <child link="wheel_right_link"/>
-    <origin xyz="0.00 -${0.23/2} 0.0250" rpy="${-M_PI/2} 0 0"/>
-  </joint>
-  <link name="wheel_right_link">
-    <visual>
-      <geometry>
-        <cylinder length="0.0206" radius="0.0350"/>
-      </geometry>
-      <origin xyz="0 0 0" rpy="0 0 0"/>
-    </visual>
-    <collision>
-      <geometry>
-        <cylinder length="0.0206" radius="0.0350"/>
-      </geometry>
-      <origin rpy="0 0 0" xyz="0 0 0"/>
-    </collision>
-    <inertial>
-      <mass value="0.01" />
-      <origin xyz="0 0 0" />
-      <inertia ixx="0.001" ixy="0.0" ixz="0.0"
-               iyy="0.001" iyz="0.0"
-               izz="0.001" />
-    </inertial>
-  </link>
-  <joint name="caster_front_joint" type="fixed">
-    <parent link="base_link"/>
-    <child link="caster_front_link"/>
-    <origin xyz="0.115 0.0 0.007" rpy="${-M_PI/2} 0 0"/>
-  </joint>
-  <link name="caster_front_link">
-    <collision>
-      <geometry>
-        <cylinder length="0.0176" radius="0.017"/>
-      </geometry>
-      <origin rpy="0 0 0" xyz="0 0 0"/>
-    </collision>
-    <inertial>
-      <mass value="0.01" />
-      <origin xyz="0 0 0" />
-      <inertia ixx="0.001" ixy="0.0" ixz="0.0"
-               iyy="0.001" iyz="0.0"
-               izz="0.001" />
-    </inertial>
-  </link>
-  <joint name="caster_back_joint" type="fixed">
-    <parent link="base_link"/>
-    <child link="caster_back_link"/>
-    <origin xyz="-0.135 0.0 0.009" rpy="${-M_PI/2} 0 0"/>
-  </joint>
-  <link name="caster_back_link">
-    <collision>
-      <geometry>
-        <cylinder length="0.0176" radius="0.017"/>
-      </geometry>
-      <origin rpy="0 0 0" xyz="0 0 0"/>
-    </collision>
-    <inertial>
-      <mass value="0.01" />
-      <origin xyz="0 0 0" />
-      <inertia ixx="0.001" ixy="0.0" ixz="0.0"
-               iyy="0.001" iyz="0.0"
-               izz="0.001" />
-    </inertial>
-  </link>
-  <gazebo reference="wheel_left_link">
-    <mu1>1.0</mu1>
-    <mu2>1.0</mu2>
-    <kp>1000000.0</kp>
-    <kd>100.0</kd>
-    <minDepth>0.001</minDepth>
-    <maxVel>1.0</maxVel>
-  </gazebo>
-  <gazebo reference="wheel_right_link">
-    <mu1>1.0</mu1>
-    <mu2>1.0</mu2>
-    <kp>1000000.0</kp>
-    <kd>100.0</kd>
-    <minDepth>0.001</minDepth>
-    <maxVel>1.0</maxVel>
-  </gazebo>
-  <gazebo reference="caster_front_link">
-    <mu1>0.0</mu1>
-    <mu2>0.0</mu2>
-    <kp>1000000.0</kp>
-    <kd>100.0</kd>
-    <minDepth>0.001</minDepth>
-    <maxVel>1.0</maxVel>
-  </gazebo>
-  <gazebo reference="caster_back_link">
-    <mu1>0.0</mu1>
-    <mu2>0.0</mu2>
-    <kp>1000000.0</kp>
-    <kd>100.0</kd>
-    <minDepth>0.001</minDepth>
-    <maxVel>1.0</maxVel>
-  </gazebo>
-  <gazebo>
-    <plugin name="differential_drive_controller" filename="libgazebo_ros_diff_drive.so">
-      <alwaysOn>true</alwaysOn>
-      <updateRate>100</updateRate>
-      <leftJoint>wheel_right_joint</leftJoint>
-      <rightJoint>wheel_left_joint</rightJoint>
-      <wheelSeparation>0.230</wheelSeparation>
-      <wheelDiameter>0.070</wheelDiameter>
-      <torque>20</torque>
-      <commandTopic>cmd_vel</commandTopic>
-      <odometryTopic>odom</odometryTopic>
-      <odometryFrame>world</odometryFrame>
-      <robotBaseFrame>base_footprint</robotBaseFrame>
-    </plugin>
-  </gazebo>
-  <!-- Kinect -->
-  <xacro:include filename="$(find cognifli_description)/cognifli_drone/urdf/kinect_camera.urdf.xacro" />
-  <xacro:kinect_camera name="kinect" parent="base_link">
-    <origin xyz="${0.178/2} 0 ${0.3/2}" rpy="0.0 0.0 0.0"/>
-  </xacro:kinect_camera>
-  <!-- Generic camera
-  <xacro:include filename="$(find cognifli_description)/cognifli_drone/urdf/generic_camera.urdf.xacro" />
-  <xacro:generic_camera name="generic_camera" parent="base_link" ros_topic="/sensors/generic_camera/image" cam_info_topic="/sensors/generic_camera/camera_info" update_rate="15" res_x="320" res_y="240" image_format="L8" hfov="75">
-    <origin xyz="${base_x_size/2-camera_link/2} 0 ${base_z_size/2 + camera_link/2}" rpy="0 0 3.14"/>
-  </xacro:generic_camera>-->
+<robot name="cognifli" xmlns:xacro="http://ros.org/wiki/xacro">
+  <xacro:include filename="$(find cognifli_description)/urdf/component_snippets.xacro" />
+  <!-- Instantiate ardrone "mechanics" -->
+  <xacro:include filename="$(find cognifli_description)/urdf/cognifli_mechanics.xacro" />
+  <!-- Instantiate a controller. -->
+  <xacro:controller_plugin_macro namespace="${namespace}" imu_sub_topic="imu" />
+  <xacro:if value="$(arg enable_mavlink_interface)">
+    <!-- Instantiate mavlink telemetry interface. -->
+    <xacro:default_mavlink_interface namespace="${namespace}" imu_sub_topic="imu" rotor_count="4" />
+  </xacro:if>
+  <!-- Mount an ADIS16448 IMU. -->
+  <xacro:default_imu namespace="${namespace}" parent_link="${namespace}/base_link" />
+  <xacro:if value="$(arg enable_ground_truth)">
+    <xacro:ground_truth_imu_and_odometry namespace="${namespace}" parent_link="${namespace}/base_link" />
+  </xacro:if>
+  <xacro:if value="$(arg enable_logging)">
+    <!-- Instantiate a logger -->
+    <xacro:bag_plugin_macro
+      namespace="${namespace}"
+      bag_file="$(arg log_file)"
+      rotor_velocity_slowdown_sim="${rotor_velocity_slowdown_sim}"
+      wait_to_record_bag="$(arg wait_to_record_bag)" />
+  </xacro:if>
 </robot>
